File: Projeto Integrador III/simulations/low_pass_filter_2/low_pass_filter_2.kicad_sch (KiCad schematic)
At the start: 8 parts, among them U1 ${SIM.PARAMS}

Commit message: PCI Finalizada V2
Parts:
- C2: value 22n -> 20n
Changed lines of the file:
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@@
 			)
 		)
-		(property "Value" "22n"
+		(property "Value" "20n"
 			(at 52.07 19.05 90)
 			(effects
