File: Projeto Integrador III/simulations/notch_filter/notch_filter.kicad_sch (KiCad schematic)
At the start: 13 parts, among them U1 ${SIM.PARAMS}, U2 ${SIM.PARAMS}

Commit message: PCI Finalizada V2
Parts:
- C1, C2: value 4u -> 20n
- C3: value 8u -> 39n
- R1, R2: value 664R -> 133k
- R3: value 332R -> 66.5k
- R5: value 3.9k -> 3.91k
